File: TerminalServer/TerminalServer.kicad_sch (KiCad schematic)
At the start: 129 parts, among them J1 RJ45_LED, J10 Conn_01x10_Pin, J11 SI-60118-F, J12 Conn_01x08_Pin, J13 503398-1892, J2 RJ45_LED, J3 RJ45_LED, J4 RJ45_LED, J5 RJ45_LED, J6 RJ45_LED, J7 USB_B, J8 Barrel_Jack_Switch, J9 Conn_PIC_ICSP_ICD, SW1 SW_Push, SW2 SW_SPDT, U1 PIC32MX795F512L-80x-PT, U10 24LC16, U11 ENC28J60x-ML, U12 ESP32-S3-WROOM-1, U2 XR32330EBERTR-F, U3 XR32330EBERTR-F, U4 XR32330EBERTR-F, U5 XR32330EBERTR-F, U6 XR32330EBERTR-F, U7 XR32330EBERTR-F, U9 TPS82130, Y1 ASEMB-8.000MHZ-LC-T, Y2 ASEMB-25.000MHZ-LC-T

Commit message: Initial firmware work
Parts:
- added R35, R36: 10k, Resistor_SMD:R_0603_1608Metric_Pad0.98x0.95mm_HandSolder, symbol Device:R_Small
- D1, D2, D3: Mouser (none) -> 78-V8PAN50-M3/I
- D4: Mouser (none) -> 604-WP914CK4GDT
- J1, J2, J3, J4, J5, J6: Mouser (none) -> 737-MTJ-88ARX1-LH
- J7: Mouser (none) -> 200-USBBSFBTHFR
- J8: Mouser (none) -> 710-694106301002
- SW2: footprint Button_Switch_THT:SW_Slide_SP3T_Straight_CK_OS103012MU1QP1 -> Library:34ASP23B4M7RT
Connections:
- net ENC_INT: now also R36.2
- net ESP_INT: now also R35.2
- net VDD: now also R35.1, R36.1

Commit message: Tie A2 of EEPROM high and move RS232 driver SHUTDOWN (now tied high) to ONLINE pin.
Connections:
- net GND: no longer U10.3 (A2)
- net U1SHTDN: now also U2.15 (*ONLINE); no longer U2.14 (*SHUTDOWN)
- net U2SHTDN: now also U3.15 (*ONLINE); no longer U3.14 (*SHUTDOWN)
- net U3SHTDN: now also U4.15 (*ONLINE); no longer U4.14 (*SHUTDOWN)
- net U4SHTDN: now also U5.15 (*ONLINE); no longer U5.14 (*SHUTDOWN)
- net U5SHTDN: now also U6.15 (*ONLINE); no longer U6.14 (*SHUTDOWN)
- net U6SHTDN: now also U7.15 (*ONLINE); no longer U7.14 (*SHUTDOWN)
- net VDD: now also U10.3 (A2), U2.14 (*SHUTDOWN), U3.14 (*SHUTDOWN), U4.14 (*SHUTDOWN), U5.14 (*SHUTDOWN), U6.14 (*SHUTDOWN), U7.14 (*SHUTDOWN); no longer U2.15 (*ONLINE), U3.15 (*ONLINE), U4.15 (*ONLINE), U5.15 (*ONLINE), U6.15 (*ONLINE), U7.15 (*ONLINE)
